File: RemoteControlLight.kicad_sch (KiCad schematic)
At the start: 5 parts, among them U1 AD009-01X

Commit message: 修改
Parts:
- C1: value C_Polarized -> 6.3v 100uF; footprint (none) -> Capacitor_THT:CP_Radial_D5.0mm_P2.00mm
- C2: footprint (none) -> Capacitor_SMD:C_0805_2012Metric
- R1: footprint (none) -> Resistor_SMD:R_0805_2012Metric
Changed lines of the file:
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@@
 			)
 		)
-		(property "Footprint" ""
+		(property "Footprint" "Capacitor_SMD:C_0805_2012Metric"
 			(at 68.8848 91.44 0)
 			(effects
@@
 			)
 		)
-		(property "Footprint" ""
+		(property "Footprint" "Resistor_SMD:R_0805_2012Metric"
 			(at 87.122 109.22 90)
 			(effects
@@
 			)
 		)
-		(property "Value" "C_Polarized"
+		(property "Value" "6.3v 100uF"
 			(at 92.71 97.4089 0)
 			(effects
@@
 			)
 		)
-		(property "Footprint" ""
+		(property "Footprint" "Capacitor_THT:CP_Radial_D5.0mm_P2.00mm"
 			(at 87.9348 91.44 0)
 			(effects
